File: PCB/measure_zero/measure_zero.kicad_sch (KiCad schematic)
At the start: 12 parts, among them J1 Conn_01x03_Pin, SW1 SW_MEC_5E, U1 ESP32-C3FH4, U2 NE555D

Commit message: afds
Parts:
- added Je1: Barrel_Jack, Connector_BarrelJack:BarrelJack_CLIFF_FC681465S_SMT_Horizontal, symbol Connector:Barrel_Jack
Changed lines of the file:
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@@
+		)
+	)
+	(symbol
+		(lib_id "Connector:Barrel_Jack")
+		(at 142.24 68.58 0)
+		(unit 1)
+		(body_style 1)
+		(exclude_from_sim no)
+		(in_bom yes)
+		(on_board yes)
+		(in_pos_files yes)
+		(dnp yes)
+		(fields_autoplaced yes)
+		(property "Reference" "Je1"
+			(at 142.24 59.69 0)
+			(show_name no)
+			(do_not_autoplace no)
+			(effects
+				(font
+					(size 1.27 1.27)
+				)
+			)
+		)
+		(property "Value" "Barrel_Jack"
+			(at 142.24 62.23 0)
+			(show_name no)
+			(do_not_autoplace no)
+			(effects
+				(font
+					(size 1.27 1.27)
+				)
+			)
+		)
+		(property "Footprint" "Connector_BarrelJack:BarrelJack_CLIFF_FC681465S_SMT_Horizontal"
+			(at 143.51 69.596 0)
+			(hide yes)
+			(show_name no)
+			(do_not_autoplace no)
+			(effects
+				(font
+					(size 1.27 1.27)
+				)
+			)
+		)
+		(property "Datasheet" ""
+			(at 143.51 69.596 0)
+			(hide yes)
+			(show_name no)
+			(do_not_autoplace no)
+			(effects
+				(font
+					(size 1.27 1.27)
+				)
+			)
+		)
+		(property "Description" "DC Barrel Jack"
+			(at 142.24 68.58 0)
+			(hide yes)
+			(show_name no)
+			(do_not_autoplace no)
+			(effects
+				(font
+					(size 1.27 1.27)
+				)
+			)
+		)
+		(pin "2"
+		)
+		(pin "1"
+		)
+		(instances
+			(project "measure_zero"
+				(path "/646a13c6-1699-4beb-a604-bf7507e93d69"
+					(reference "Je1")
+					(unit 1)
+				)
+			)
 		)
 	)
