File: PCB/measure_zero/measure_zero.kicad_pcb (KiCad board)
At the start: 2 copper layers, 300 x 30 mm, 12 parts

Commit message: Update measure_zero.kicad_pcb
Other:
- outline, holes or cut-outs redrawn
- board text added: "Measure Zero"
- board text removed: "20mm"
Changed lines of the file:
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@@
 	)
 	(gr_circle
-		(center 200.5 -3.5)
-		(end 203 -3.5)
+		(center 211.5 -3.5)
+		(end 214 -3.5)
 		(stroke
 			(width 0.1)
@@
 	)
 	(gr_circle
-		(center 211.5 -3.5)
-		(end 215.5 -3.5)
+		(center 222.5 -3.5)
+		(end 226.5 -3.5)
 		(stroke
 			(width 0.1)
@@
 	)
 	(gr_circle
-		(center 226 -3.5)
-		(end 231 -3.5)
+		(center 237 -3.5)
+		(end 242 -3.5)
 		(stroke
 			(width 0.1)
@@
 	)
 	(gr_circle
-		(center 247 -3.5)
-		(end 254.5 -3.5)
+		(center 256.5 -3.5)
+		(end 264 -3.5)
 		(stroke
 			(width 0.1)
@@
 		(layer "Edge.Cuts")
 	)
-	(gr_circle
-		(center 275 -3.5)
-		(end 285 -3.5)
-		(stroke
-			(width 0.1)
-			(type solid)
-		)
-		(fill no)
-		(layer "Edge.Cuts")
-	)
 	(gr_text " 0\n"
 		(at 10 -15 0)
@@
 		)
 	)
+	(gr_text "Measure Zero"
+		(at 267 -3.5 0)
+		(layer "F.Cu")
+		(effects
+			(font
+				(size 4 4)
+				(thickness 0.8)
+				(bold yes)
+			)
+			(justify left bottom)
+		)
+	)
 	(gr_text "1mm"
 		(at 142 -11 0)
@@
 	)
 	(gr_text "5mm"
-		(at 204.5 -6.5 0)
+		(at 215.5 -6.5 0)
 		(layer "F.SilkS")
 		(effects
@@
 	)
 	(gr_text "8mm"
-		(at 216.5 -7.5 0)
+		(at 227.5 -7.5 0)
 		(layer "F.SilkS")
 		(effects
@@
 	)
 	(gr_text "10mm"
-		(at 231 -9 0)
+		(at 242 -9 0)
 		(layer "F.SilkS")
 		(effects
@@
 	)
 	(gr_text "15mm"
-		(at 255 -10.5 0)
-		(layer "F.SilkS")
-		(effects
-			(font
-				(size 1 1)
-				(thickness 0.1)
-			)
-			(justify top)
-		)
-	)
-	(gr_text "20mm"
-		(at 287 -9.5 0)
+		(at 264.5 -10.5 0)
 		(layer "F.SilkS")
 		(effects
@@
 			)
 			(justify left bottom)
+		)
+	)
+	(gr_text "Measure Zero"
+		(at 267 -3.5 0)
+		(layer "F.SilkS")
+		(effects
+			(font
+				(size 4 4)
+				(thickness 0.4)
+			)
+			(justify left bottom)

Commit message: afds
Parts:
- added Barrel Jack: Barrel_Jack, Connector_BarrelJack:BarrelJack_CLIFF_FC681465S_SMT_Horizontal, F.Cu at (66.5, -1.00)
- moved USB A 2.06 mm to (27.0, -5.89)
- moved USB C 2.00 mm to (42.2, -8.12)
- moved QFN32 1.75 mm to (53.2, -10.5)
Other:
- outline, holes or cut-outs redrawn
- board text added: "135º"
- board text added: "Stencils"
- board text added: "rev 1"

Commit message: tweeks
Parts:
- moved USB A 0.55 mm to (26.4, -5.89)
Routing:
- net (no net): track 0.00 -> 27.0 mm
- net unconnected-(USB2-VCC-Pad1): track 0.00 -> 25.0 mm
- net unconnected-(Je1-Pad1): track 0.00 -> 15.0 mm
Other:
- board text added: "01"
- board text added: "02"
Changed lines of the file:
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@@
 		(capping no)
 		(filling no)
-		(zone_defaults)
 		(pcbplotparams
 			(layerselection 0x00000000_00000000_55555555_5755f5ff)
@@
 	(footprint "lcsc:USB-A-TH_10.0QHHTZB6.3"
 		(layer "F.Cu")
-		(at 27 -5.89 180)
+		(at 26.45 -5.89 180)
 		(property "Reference" "USB A"
-			(at 0 -7.11 0)
+			(at 6.95 -4.39 0)
 			(layer "F.SilkS")
 			(effects
@@
 				(font
 					(size 1.27 1.27)
+					(thickness 0.15)
 				)
 			)
@@
 				(font
 					(size 1.27 1.27)
+					(thickness 0.15)
 				)
 			)
@@
 				(font
 					(size 1.27 1.27)
+					(thickness 0.15)
 				)
 			)
@@
 		(layer "F.Cu")
 	)
+	(gr_line
+		(start 34 -19)
+		(end 34 -20)
+		(stroke
+			(width 0.1)
+			(type default)
+		)
+		(layer "F.Cu")
+	)
+	(gr_line
+		(start 35 -18)
+		(end 35 -20)
+		(stroke
+			(width 0.1)
+			(type default)
+		)
+		(layer "F.Cu")
+	)
 	(gr_rect
-		(start 33 -1.5)
-		(end 58 -1.4)
+		(start 35 -2.1)
+		(end 58 -2)
 		(stroke
 			(width 0)
@@
 	)
 	(gr_rect
-		(start 33 -0.85)
-		(end 58 -0.65)
+		(start 35 -1.45)
+		(end 58 -1.25)
 		(stroke
 			(width 0)
@@
 	)
 	(gr_rect
-		(start 33 0.15)
-		(end 58 0.45)
+		(start 35 -0.45)
+		(end 58 -0.15)
 		(stroke
 			(width 0)
@@
 	)
 	(gr_rect
-		(start 33 1)
-		(end 58 1.5)
+		(start 35 0.4)
+		(end 58 0.9)
 		(stroke
 			(width 0)
@@
 	)
 	(gr_rect
-		(start 33 2)
-		(end 58 3)
+		(start 35 1.4)
+		(end 58 2.4)
 		(stroke
 			(width 0)
@@
 	)
 	(gr_rect
-		(start 33 3.5)
-		(end 58 5.5)
+		(start 35 2.9)
+		(end 58 4.9)
 		(stroke
 			(width 0)
@@
 	)
 	(gr_line
-		(start 34 -19)
-		(end 34 -20)
-		(stroke
-			(width 0.1)
-			(type default)
-		)
-		(layer "F.Cu")
-	)
-	(gr_line
-		(start 35 -18)
-		(end 35 -20)
-		(stroke
-			(width 0.1)
-			(type default)
-		)
-		(layer "F.Cu")
-	)
-	(gr_line
 		(start 35.56 10.16)
 		(end 35.56 6.985)
@@
 		)
 	)
+	(gr_text "05\n\n"
+		(at 30 3.5 0)
+		(layer "F.SilkS")
+		(effects
+			(font
+				(size 1 1)
+				(thickness 0.1)
+			)
+			(justify left bottom)
+		)
+	)
+	(gr_text "1\n"
+		(at 30.5 3.5 0)
+		(layer "F.SilkS")
+		(effects
+			(font
+				(size 1 1)
+				(thickness 0.1)
+			)
+			(justify left bottom)
+		)
+	)
+	(gr_text "02\n"
+		(at 32 -1 0)
+		(layer "F.SilkS")
+		(effects
+			(font
+				(size 1 1)
+				(thickness 0.1)
+			)
+			(justify left bottom)
+		)
+	)
+	(gr_text "03\n"
+		(at 32 0.5 0)
+		(layer "F.SilkS")
+		(effects
+			(font
+				(size 1 1)
+				(thickness 0.1)
+			)
+			(justify left bottom)
+		)
+	)
+	(gr_text "2"
+		(at 33.5 4.5 0)
+		(layer "F.SilkS")
+		(effects
+			(font
+				(size 1 1)
+				(thickness 0.1)
+			)
+			(justify left bottom)
+		)
+	)
+	(gr_text "01"
+		(at 34 -3.5 0)
+		(layer "F.SilkS")
+		(effects
+			(font
+				(size 1 1)
+				(thickness 0.1)
+			)
+			(justify left bottom)
+		)
+	)
 	(gr_text "135º"
 		(at 130.5 -9.5 0)
@@
 		)
 	)
-	(gr_text "M2"
-		(at 174 -2.5 0)
+	(gr_text "1.5"
+		(at 117.5 1 0)
 		(layer "F.SilkS")
 		(effects
@@
 		)
 	)
-	(gr_text "M2.5"
-		(at 179 -2.5 0)
+	(gr_text "03"
+		(at 118 -14 0)
 		(layer "F.SilkS")
 		(effects
@@
 		)
 	)
-	(gr_text "M3"
-		(at 184 -2.5 0)
+	(gr_text "05"
+		(at 118 -11 0)
 		(layer "F.SilkS")
 		(effects
@@
 		)
 	)
-	(gr_text "M4"
-		(at 190 -2.5 0)
+	(gr_text "06"
+		(at 118 -8 0)
 		(layer "F.SilkS")
 		(effects
@@
 		)
 	)
-	(gr_text "5mm"
-		(at 208 -6.5 0)
+	(gr_text "08"
+		(at 118 -5 0)
 		(layer "F.SilkS")
 		(effects
@@
 		)
 	)
-	(gr_text "8mm"
-		(at 220 -7.5 0)
+	(gr_text "1"
+		(at 118 -2 0)
 		(layer "F.SilkS")
 		(effects
@@
 		)
 	)
-	(gr_text "10mm"
-		(at 234.5 -9 0)
+	(gr_text "2\n"
+		(at 118 4 0)
 		(layer "F.SilkS")
 		(effects
@@
 		)
 	)
-	(gr_text "15mm"
-		(at 257 -10.5 0)
+	(gr_text "M2"
+		(at 174 -2.5 0)
 		(layer "F.SilkS")
 		(effects
@@
 		)
 	)
-	(gr_text "5mm"
-		(at 15 -8.5 0)
+	(gr_text "M2.5"
+		(at 179 -2.5 0)
 		(layer "F.SilkS")
 		(effects
@@
 				(thickness 0.1)
 			)
+			(justify top)
 		)
 	)
-	(gr_text "03"
-		(at 118 -13.5 270)
+	(gr_text "M3"
+		(at 184 -2.5 0)
 		(layer "F.SilkS")
 		(effects
@@
 		)
 	)
-	(gr_text "05"
-		(at 118 -10.5 270)
+	(gr_text "M4"
+		(at 190 -2.5 0)
 		(layer "F.SilkS")
 		(effects
@@
 		)
 	)
-	(gr_text "06"
-		(at 118 -7.5 270)
+	(gr_text "5mm"
+		(at 208 -6.5 0)
 		(layer "F.SilkS")
 		(effects
@@
 		)
 	)
-	(gr_text "08"
-		(at 118 -4.5 270)
+	(gr_text "8mm"
+		(at 220 -7.5 0)
 		(layer "F.SilkS")
 		(effects
@@
 		)
 	)
-	(gr_text "1"
-		(at 118 -1.5 270)
+	(gr_text "10mm"
+		(at 234.5 -9 0)
 		(layer "F.SilkS")
 		(effects
@@
 		)
 	)
-	(gr_text "1.5"
-		(at 118 1.5 270)
+	(gr_text "15mm"
+		(at 257 -10.5 0)
 		(layer "F.SilkS")
 		(effects
@@
 		)
 	)
-	(gr_text "2\n"
-		(at 118 4.5 270)
+	(gr_text "5mm"
+		(at 15 -8.5 0)
 		(layer "F.SilkS")
 		(effects
@@
 				(thickness 0.1)
 			)
-			(justify top)
 		)
 	)
-	(gr_text "Stencils"
-		(at 128.5 -12 0)
+	(gr_text "Vias"
+		(at 121.5 -12 0)
 		(layer "F.SilkS")
 		(effects
@@
 		)
 	)
-	(gr_text "Screws"
-		(at 172 -11 0)
+	(gr_text "Stencils"
+		(at 128.5 -12 0)
 		(layer "F.SilkS")
 		(effects
@@
 		)
 	)
-	(gr_text "Holes"
-		(at 201 -12 0)
+	(gr_text "Screws"
+		(at 172 -11 0)
 		(layer "F.SilkS")
 		(effects
@@
 		)
 	)
-	(gr_text "Vias"
-		(at 122 -14 270)
+	(gr_text "Holes"
+		(at 201 -12 0)
 		(layer "F.SilkS")
 		(effects
@@
 		)
 	)
+	(segment
+		(start 46.5 0.65)
+		(end 33.85 0.65)
+		(width 0.5)
+		(layer "F.Cu")
+		(net "")
+	)
+	(segment
+		(start 46.5 -0.3)
+		(end 34.3 -0.3)
+		(width 0.3)
+		(layer "F.Cu")
+		(net "")
+	)
+	(segment
+		(start 34.3 -0.3)
+		(end 34 0)
+		(width 0.3)
+		(layer "F.Cu")
+		(net "")
+	)
+	(segment
+		(start 33 1.5)
+		(end 32.5 1.5)
+		(width 0.5)
+		(layer "F.Cu")
+		(net "")
+	)
+	(segment
+		(start 33.85 0.65)
+		(end 33 1.5)
+		(width 0.5)
+		(layer "F.Cu")
+		(net "")
+	)
 	(via
 		(at 120 -1.5)
@@
 		(net "")
 	)
+	(segment
+		(start 34.5 -2.5)
+		(end 34.5 -3)
+		(width 0.1)
+		(layer "F.Cu")
+		(net "unconnected-(USB2-VCC-Pad1)")
+	)
+	(segment
+		(start 46.5 -2.05)
+		(end 34.95 -2.05)
+		(width 0.1)
+		(layer "F.Cu")
+		(net "unconnected-(USB2-VCC-Pad1)")
+	)
+	(segment
+		(start 46.5 -1.35)
+		(end 34.15 -1.35)
+		(width 0.2)
+		(layer "F.Cu")
+		(net "unconnected-(USB2-VCC-Pad1)")
+	)
+	(segment
+		(start 34.95 -2.05)
+		(end 34.5 -2.5)
+		(width 0.1)
+		(layer "F.Cu")
+		(net "unconnected-(USB2-VCC-Pad1)")
+	)
+	(segment
+		(start 46.5 1.9)
+		(end 34.1 1.9)
+		(width 1)
+		(layer "F.Cu")
+		(net "unconnected-(Je1-Pad1)")
+	)
+	(segment
+		(start 34.1 1.9)
+		(end 33 3)
+		(width 1)
+		(layer "F.Cu")
+		(net "unconnected-(Je1-Pad1)")
+	)
+	(segment
+		(start 33 3)
+		(end 32 3)
+		(width 1)
+		(layer "F.Cu")
+		(net "unconnected-(Je1-Pad1)")
+	)
 	(embedded_fonts no)

Commit message: masking
Routing:
- net unconnected-(SW1-Pad2): vias 0 -> 1
- net unconnected-(R1-Pad2): vias 0 -> 2
- net unconnected-(R1-Pad1): vias 0 -> 1
- net unconnected-(D1-A-Pad2): vias 0 -> 1
- net (no net): vias 11 -> 6
